Commit message: change config

File: src/ua_simulator/urdf/DIODE_robot.urdf.xacro (robot description, xacro)
@@ -190,11 +190,3 @@
       xyz="0 0 0" />
   </joint>
-  <xacro:arg name="gpu" default="false"/>
-  <xacro:property name="gpu" value="$(arg gpu)" />
-  <xacro:arg name="organize_cloud" default="false"/>
-  <xacro:property name="organize_cloud" value="$(arg organize_cloud)" />
-  <xacro:include filename="$(find ua_simulator)/urdf/HDL-32E.urdf.xacro"/>
-  <xacro:HDL-32E parent="$(arg robot_name)/base_link" name="velodyne2" topic="/velodyne_points2" organize_cloud="${organize_cloud}" hz="10" samples="220" gpu="${gpu}">
-    <origin xyz="0.053735 -0.0017816 0.12" rpy="0 0 0" />
-  </xacro:HDL-32E>
 </robot>
